File: pcb/hack_matrix.kicad_sch (KiCad schematic)
At the start: 16 parts, among them J1 USB_C_Receptacle_USB2.0_16P, J2 Screw_Terminal_01x02, SW2 SW_Push, U1 SN74AHCT245PWR, U3 XC6206P332MR, U4 ESP32-S2-MINI-2, U5 SN74AHCT245PWR

Commit message: esp32-s2 -> esp32-s3
Parts:
- removed U4: ESP32-S2-MINI-2, ESP32-S2-MINI-2:XCVR_ESP32-S2-MINI-2, symbol ESP32-S2-MINI-2:ESP32-S2-MINI-2
- added U6: ESP32-S3-MINI-1-N8, RF_Module:ESP32-S2-MINI-1, symbol RF_Module:ESP32-S3-MINI-1
Connections:
- net +3V3: now also U6.3 (3V3), U6.45 (EN)
- net A: now also U6.12 (IO8)
- net B: now also U6.11 (IO7)
- net B1: now also U6.7 (IO3)
- net B2: now also U6.10 (IO6)
- net C: now also U6.14 (IO10)
- net CLK: now also U6.16 (IO12)
- net D: now also U6.13 (IO9)
- net D+: now also U6.24 (USB_D+)
- net D-: now also U6.23 (USB_D-)
- net G1: now also U6.6 (IO2)
- net G2: now also U6.8 (IO4)
- net GND: now also U6.1 (GND), U6.2 (GND), U6.42 (GND), U6.43 (GND), U6.46 (GND), U6.47 (GND), U6.48 (GND), U6.49 (GND), U6.50 (GND), U6.51 (GND), U6.52 (GND), U6.53 (GND), U6.54 (GND), U6.55 (GND), U6.56 (GND), U6.57 (GND), U6.58 (GND), U6.59 (GND), U6.60 (GND), U6.61 (GND), U6.62 (GND), U6.63 (GND), U6.64 (GND), U6.65 (GND)
- net GPIO0: now also U6.4 (IO0)
- net OE-: now also U6.17 (IO13)
- net R1: now also U6.5 (IO1)
- net R2: now also U6.9 (IO5)
- net STROBE: now also U6.15 (IO11)
- no-connect marks 24 -> 28
Other:
- moved on the sheet: J2
